Commit message: Refactor SO101 task environment and motion planning for lift task
- Integrated SO101TaskEnv into the task planner for better environment management.
- Removed redundant functions and debug code related to gripper width.
- Simplified the grasp pose calculation and motion execution for the lift task.
- Updated the approach to reach and grasp poses to align with SO101's requirements.
- Enhanced the overall structure and readability of the motion planning code.

File: assets/SO101/so101.urdf (robot description, URDF)
Before this commit: robot so101_new_calib, 9 links, 8 joints
Links:
- removed link gripper_frame_link
- added link gripper_link_tip; visual sphere radius=0.01
- added link moving_jaw_so101_v1_link_tip; visual sphere radius=0.01
- link camera_link: mass 1e-6 -> 0
- link gripper_link: geometry collision mesh filename=assets/Fixed_Jaw_part1.ply; collision mesh filename=assets/Fixed_Jaw_part2.ply
- link moving_jaw_so101_v1_link: geometry collision mesh filename=assets/Moving_Jaw_part1.ply; collision mesh filename=assets/Moving_Jaw_part2.ply
Joints:
- removed joint gripper_frame_joint
- added joint gripper_link_tip_joint: type fixed, parent gripper_link, child gripper_link_tip, origin xyz=-0.01 0 0.097 rpy=0 0 0
- added joint moving_jaw_so101_v1_link_tip_joint: type fixed, parent moving_jaw_so101_v1_link, child moving_jaw_so101_v1_link_tip, origin xyz=-0.01 -0.073 0.02 rpy=0 0 0
- joint elbow_flex: limit lower=-1.69 upper=1.69 effort=10 velocity=10 -> lower=-1.69 upper=1.69 effort=0 velocity=0
- joint gripper: limit lower=-0.174533 upper=1.74533 effort=10 velocity=10 -> lower=-0.174533 upper=1.74533 effort=0 velocity=0; origin xyz=0.0202 0.0188 -0.0234 rpy=1.5708 -5.24284e-08 -1.41553e-15 -> xyz=0.0202 -0.0188 0.0234 rpy=-1.5708 -5.24284e-08 -1.41553e-15
- joint gripper_camera_joint: origin xyz=0.0 -0.0383 -0.0680 rpy=-3.14159 1.1344639 1.5707968 -> xyz=0.0 -0.0383 0.0680 rpy=3.14159 -2.0055361 -1.5707968
- joint shoulder_lift: limit lower=-1.74533 upper=1.74533 effort=10 velocity=10 -> lower=-1.74533 upper=1.74533 effort=0 velocity=0
- joint shoulder_pan: limit lower=-1.91986 upper=1.91986 effort=10 velocity=10 -> lower=-1.91986 upper=1.91986 effort=0 velocity=0
- joint wrist_flex: limit lower=-1.65806 upper=1.65806 effort=10 velocity=10 -> lower=-1.65806 upper=1.65806 effort=0 velocity=0
- joint wrist_roll: limit lower=-2.74385 upper=2.84121 effort=10 velocity=10 -> lower=-2.74385 upper=2.84121 effort=0 velocity=0; origin xyz=5.55112e-17 -0.0611 0.0181 rpy=1.5708 0.0486795 3.14159 -> xyz=5.55112e-17 -0.0611 0.0181 rpy=-1.5708 0.0486795 3.14159
